File: ESC.sch (EAGLE design)
At the start: 45 parts, among them M1 IRF3205, M2 IRF3205, M3 IRF3205, M4 IRF3205, M5 IRF3205, M6 IRF3205

Commit message: Board Layout v1 final
Parts:
- C10, C2, C3, C4, C7: device TRANS_IRF3205SPBF:CAPACITORSMALL -> TRANS_IRF3205SPBF:CAPACITOR
- C11, C12, C5, C6, C8, C9: device TRANS_IRF3205SPBF:CAPACITORCERAMIC -> TRANS_IRF3205SPBF:CAPACITOR
- R1, R10, R11, R12, R4, R5, R6, R7, R8, R9: device TRANS_IRF3205SPBF:RESISTOR -> TRANS_IRF3205SPBF:RESISTOR0805
Connections:
- net N$24 renamed M6_G
- new net IN_V: C2.ANODE, R2.2, R3.2, U1.IN
- net 5V_OUT: now also R1.2
- net A_HI: now also NANO.D6; no longer NANO.D2
- net A_LO: now also NANO.D7; no longer NANO.D3
- net C_HI: now also NANO.D2; no longer NANO.D6
- net C_LO: now also NANO.D3; no longer NANO.D7
- net POWER: no longer C2.ANODE, R1.2, R2.2, R3.2, U1.IN
Other:
- moved on the sheet: LED, R1, R2, TC1, TC2, TC3
